File: PCB/DynaLab/DynaLab.kicad_pcb (KiCad board)
At the start: 2 copper layers, 150 x 80 mm, 86 parts, among them J1 USB_C_Receptacle_USB2.0_16P, SW1 BOOT, SW2 REC/STOP, SW3 RESET, U1 LM393, U10 74AHCT125, U11 ITR8307-S17-TR8, U12 ITR8307-S17-TR8, U14 RP2040, U15 AMS1117-3.3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

Commit message: v0 routing complete - no errs
Parts:
- added C22: 100n, Capacitor_SMD:C_0603_1608Metric, B.Cu at (369.1, 275.6)
- added F1: PolyFuse 1A Trip, Resistor_SMD:R_1206_3216Metric, B.Cu at (310.8, 268.2)
- added U13: USBLC6-2SC6, Package_TO_SOT_SMD:SOT-23-6, B.Cu at (319.1, 273.2)
- added kibuzzard-6930ADF3: G***, kibuzzard-6930ADF3, F.Cu at (385.2, 267.4)
- added kibuzzard-6930AE56: G***, kibuzzard-6930AE56, B.Cu at (339.2, 292.4)
- added kibuzzard-6930AEF9: G***, kibuzzard-6930AEF9, B.Cu at (401.6, 222.0)
- added kibuzzard-6930AF86: G***, kibuzzard-6930AF86, F.Cu at (355.1, 282.0)
- added kibuzzard-6930AFAB: G***, kibuzzard-6930AFAB, F.Cu at (339.2, 265.2)
- added kibuzzard-6930BD82: G***, kibuzzard-6930BD82, F.Cu at (314.0, 271.5)
- added kibuzzard-6930BD9C: G***, kibuzzard-6930BD9C, F.Cu at (385.2, 283.0)
- D2: moved to F.Cu
- R14, R19, R8: moved to B.Cu
- TP1, TP2, TP3, TP4, TP5, TP6: footprint TestPoint:TestPoint_THTPad_1.5x1.5mm_Drill0.7mm -> TestPoint:TestPoint_Pad_D1.5mm
- moved C11 59.6 mm to (306.1, 224.4), turned to 90 degrees
- moved C18 58.8 mm to (303.8, 223.4), turned to 90 degrees
- moved C14 58.6 mm to (307.8, 226.7), turned to 90 degrees
- moved C10 57.4 mm to (311.8, 232.3), turned to 0 degrees
- moved Y1 56.4 mm to (300.8, 223.4), turned to 0 degrees
- moved R3 55.3 mm to (369.1, 272.2), turned to 180 degrees
- moved R2 55.3 mm to (369.1, 273.8), turned to 0 degrees
- moved R27 54.8 mm to (302.8, 226.1), turned to 0 degrees
- moved C15 54.5 mm to (311.8, 235.8), turned to 0 degrees
- moved C17 54.2 mm to (297.6, 223.3), turned to 90 degrees
- moved C9 53.3 mm to (311.8, 237.3), turned to 0 degrees
- moved C7 50.1 mm to (310.8, 240.1), turned to -90 degrees
- moved U14 50.0 mm to (305.7, 233.3), turned to 0 degrees
- moved C6 48.3 mm to (309.3, 240.1), turned to -90 degrees
- moved R32 47.1 mm to (322.0, 279.0), turned to 0 degrees
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Connections:
- J1 pad A4: +5V -> VBUS
- J1 pad A6: /USB_D+ -> /USB_D_RAW+
- J1 pad A7: /USB_D- -> /USB_D_RAW-
- J1 pad A9: +5V -> VBUS
- J1 pad B4: +5V -> VBUS
- J1 pad B6: /USB_D+ -> /USB_D_RAW+
- J1 pad B7: /USB_D- -> /USB_D_RAW-
- J1 pad B9: +5V -> VBUS
- U14 pad 11: /LED_REC -> unconnected-(U14-GPIO8-Pad11)
- U14 pad 12: /SW_REC -> unconnected-(U14-GPIO9-Pad12)
- U14 pad 27: /PHOTO_A -> unconnected-(U14-GPIO16-Pad27)
- U14 pad 28: /PHOTO_B -> unconnected-(U14-GPIO17-Pad28)
- U14 pad 29: /PHOTO_C -> /7SEG_CLK
- U14 pad 30: unconnected-(U14-GPIO19-Pad30) -> /7SEG_DATA
- U14 pad 31: unconnected-(U14-GPIO20-Pad31) -> /7SEG_~{CS}
- U14 pad 32: unconnected-(U14-GPIO21-Pad32) -> /SW_REC
- U14 pad 36: unconnected-(U14-GPIO24-Pad36) -> /LED_REC
- U14 pad 37: unconnected-(U14-GPIO25-Pad37) -> /PHOTO_C
- U14 pad 38: unconnected-(U14-GPIO26_ADC0-Pad38) -> /PHOTO_A
- U14 pad 39: unconnected-(U14-GPIO27_ADC1-Pad39) -> /PHOTO_B
- U14 pad 4: /7SEG_CLK -> unconnected-(U14-GPIO2-Pad4)
- U14 pad 5: /7SEG_DATA -> unconnected-(U14-GPIO3-Pad5)
- U14 pad 7: /7SEG_~{CS} -> unconnected-(U14-GPIO5-Pad7)
Routing:
- net +5V: track 0.00 -> 217.4 mm, vias 0 -> 2
- net /SW_REC: track 0.00 -> 133.2 mm, vias 0 -> 1
- net /LED_REC: track 0.00 -> 123.5 mm, vias 0 -> 2
- net /~{RESET}: track 0.00 -> 119.4 mm, vias 0 -> 1
- net GND: track 25.2 -> 135.3 mm, vias 15 -> 34
- net /7SEG_~{CS}: track 0.00 -> 108.6 mm
- net /7SEG_CLK: track 0.00 -> 104.6 mm
- net /7SEG_DATA: track 0.00 -> 102.9 mm, vias 0 -> 2
- net /PHOTO_B: track 0.00 -> 49.7 mm, vias 0 -> 2
- net /PHOTO_C: track 0.00 -> 47.1 mm, vias 0 -> 2
- net Net-(U8-LOAD): track 0.00 -> 43.5 mm
- net /PHOTO_A: track 0.00 -> 40.0 mm, vias 0 -> 2
- net /DIG2: track 0.00 -> 38.8 mm, vias 0 -> 1
- net /V_REF: track 0.00 -> 35.5 mm
- net /DIG1: track 0.00 -> 32.9 mm, vias 0 -> 1
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- added copper zone on B.Cu, net VBUS
Other:
- outline, holes or cut-outs redrawn
- board text added: "Boot"

Commit message: v01
Parts:
- removed kibuzzard-6930AE56: G***, kibuzzard-6930AE56
- removed kibuzzard-6930AEF9: G***, kibuzzard-6930AEF9
- added G***: LOGO, LOGO, B.Cu at (384.2, 236.3)
- added H10: SMTSO3040, Footprints:MountingHole_SMTSO3030_3.2mm_M3, F.Cu at (268.2, 291.0)
- added H11: SMTSO3040, Footprints:MountingHole_SMTSO3030_3.2mm_M3, F.Cu at (268.2, 260.0)
- added H12: SMTSO3040, Footprints:MountingHole_SMTSO3030_3.2mm_M3, F.Cu at (410.2, 260.0)
- added H5: SMTSO3030, Footprints:MountingHole_SMTSO3030_3.2mm_M3, B.Cu at (271.8, 250.0)
- added H6: SMTSO3030, Footprints:MountingHole_SMTSO3030_3.2mm_M3, B.Cu at (406.8, 250.0)
- added H7: SMTSO3030, Footprints:MountingHole_SMTSO3030_3.2mm_M3, B.Cu at (271.8, 220.0)
- added H8: SMTSO3030, Footprints:MountingHole_SMTSO3030_3.2mm_M3, B.Cu at (406.8, 220.0)
- added H9: SMTSO3040, Footprints:MountingHole_SMTSO3030_3.2mm_M3, F.Cu at (410.2, 291.0)
- added kibuzzard-69310180: G***, kibuzzard-69310180, B.Cu at (384.2, 228.3)
- added kibuzzard-69310240: G***, kibuzzard-69310240, B.Cu at (384.2, 244.0)
- added kibuzzard-69310248: G***, kibuzzard-69310248, B.Cu at (384.2, 246.0)
- H1, H2, H3, H4: value MountingHole -> SMTSO3030; moved to B.Cu
- SW1: moved to B.Cu
- moved G*** 112.8 mm to (390.6, 258.9)
- moved SW1 23.7 mm to (283.2, 238.8), turned to 0 degrees
- moved D1 4.30 mm to (376.8, 285.5)
- moved R26 4.30 mm to (373.1, 285.5)
- moved SW2 4.30 mm to (391.8, 283.0)
- moved SW3 4.30 mm to (391.8, 267.5)
- moved kibuzzard-6930ADF3 4.30 mm to (381.8, 269.9)
- moved kibuzzard-6930BD9C 4.30 mm to (381.8, 285.5)
- moved H1 0.94 mm to (316.8, 250.0), turned to -90 degrees
- moved H2 0.94 mm to (316.8, 220.0), turned to -90 degrees
- moved H3 0.94 mm to (361.8, 250.0), turned to -90 degrees
- moved H4 0.94 mm to (361.8, 220.0), turned to -90 degrees
Routing:
- net /~{BOOT}: track 31.7 -> 3.36 mm, vias 1 -> 0
- net /LED_REC: track 123.5 -> 105.0 mm
- net GND: track 135.3 -> 138.5 mm
- net +5V: track 217.4 -> 215.8 mm
- net /~{RESET}: track 119.4 -> 120.8 mm
- net /SW_REC: track 133.2 -> 132.0 mm
Other:
- outline, holes or cut-outs redrawn
