File: PCB/DynaLab/DynaLab.kicad_sch (KiCad schematic)
At the start: 85 parts, among them J1 USB_C_Receptacle_USB2.0_16P, SW1 BOOT, SW2 REC/STOP, SW3 RESET, U1 LM393, U10 74AHCT125, U11 ITR8307-S17-TR8, U12 ITR8307-S17-TR8, U14 RP2040, U15 AMS1117-3.3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

Commit message: v0 routing complete - no errs
Parts:
- added C22: 100n, Capacitor_SMD:C_0603_1608Metric, symbol Device:C
- added F1: PolyFuse 1A Trip, Resistor_SMD:R_1206_3216Metric, symbol Device:Polyfuse
- added U13: USBLC6-2SC6, Package_TO_SOT_SMD:SOT-23-6, symbol Power_Protection:USBLC6-2SC6
- TP1, TP2, TP3, TP4, TP5, TP6: footprint TestPoint:TestPoint_THTPad_1.5x1.5mm_Drill0.7mm -> TestPoint:TestPoint_Pad_D1.5mm
Connections:
- net +5V: now also C22.1, F1.2; no longer J1.A4 (VBUS), J1.A9 (VBUS), J1.B4 (VBUS), J1.B9 (VBUS)
- net 7SEG_CLK: now also U14.29 (GPIO18); no longer U14.4 (GPIO2)
- net 7SEG_DATA: now also U14.30 (GPIO19); no longer U14.5 (GPIO3)
- net 7SEG_~{CS}: now also U14.31 (GPIO20); no longer U14.7 (GPIO5)
- net GND: now also C22.2, U13.2 (GND)
- net LED_REC: now also U14.36 (GPIO24); no longer U14.11 (GPIO8)
- net PHOTO_A: now also U14.38 (GPIO26_ADC0); no longer U14.27 (GPIO16)
- net PHOTO_B: now also U14.39 (GPIO27_ADC1); no longer U14.28 (GPIO17)
- net PHOTO_C: now also U14.37 (GPIO25); no longer U14.29 (GPIO18)
- net SW_REC: now also U14.32 (GPIO21); no longer U14.12 (GPIO9)
- net USB_D+: now also U13.4 (I/O2); no longer J1.A6 (D+), J1.B6 (D+)
- net USB_D-: now also U13.6 (I/O1); no longer J1.A7 (D-), J1.B7 (D-)
- new net USB_D_RAW+: J1.A6 (D+), J1.B6 (D+), U13.3 (I/O2)
- new net USB_D_RAW-: J1.A7 (D-), J1.B7 (D-), U13.1 (I/O1)
- new net VBUS: F1.1, J1.A4 (VBUS), J1.A9 (VBUS), J1.B4 (VBUS), J1.B9 (VBUS), U13.5 (VBUS)
Other:
- moved on the sheet: C19, C20, D1, D2, J1, R26, R28, R29, R30, R31, R32, SW2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

Commit message: v01
Parts:
- added H10, H11, H12, H9: SMTSO3040, Footprints:MountingHole_SMTSO3030_3.2mm_M3, symbol Mechanical:MountingHole
- added H5, H6, H7, H8: SMTSO3030, Footprints:MountingHole_SMTSO3030_3.2mm_M3, symbol Mechanical:MountingHole
- D1: LCSC Part # C965804 -> C965799
- D2: LCSC Part # (none) -> C965804
- H1, H2, H3, H4: value MountingHole -> SMTSO3030
- R26: value 10k -> 220
- R30: value 10k -> 1k
- U14: LCSC Part # (none) -> C2040
- U15: LCSC Part # (none) -> C6186
- U16: LCSC Part # (none) -> C82317
Other:
- note added: "3-digit 7-Segment Display"
- note added: "Components reused to optimise BOM. Use 1V reference if desired"
- note added: "M3x3mm threaded standoffs"
- note added: "M3x4mm threaded standoffs"
- note added: "Optical encoder & Signal conditioning"
- note added: "USB Connection, Power Regulation"
- note removed: "ToDo: audit LED colour/brightness & LCSC #"
- moved on the sheet: C1, C10, C11, C12, C13, C14, C15, C16, C17, C18, C19, C2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
