File: PCB/main-board/main-board.kicad_pcb (KiCad board)
At the start: 2 copper layers, 185 x 82 mm, 114 parts, among them J1 USB_C_Receptacle_USB2.0_16P, SW1 BOOT, SW2 REC/STOP, SW3 RESET, U1 LM393, U10 74AHCT125, U11 ITR8307-S17-TR8, U12 ITR8307-S17-TR8, U13 USBLC6-2SC6, U14 RP2040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

Commit message: update 7seg display (symbol, footprint, 3Dpackage), README
Parts:
- U5, U6, U7: footprint Footprints:GS3011A -> Footprints:GS3011
