File: PCB/main-board/main-board.kicad_sch (KiCad schematic)
At the start: 94 parts, among them J1 USB_C_Receptacle_USB2.0_16P, SW1 BOOT, SW2 REC/STOP, SW3 RESET, U1 LM393, U10 74AHCT125, U11 ITR8307-S17-TR8, U12 ITR8307-S17-TR8, U13 USBLC6-2SC6, U14 RP2040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

Commit message: rename main PCB project to "main-board"
Parts:
- U5, U6, U7: symbol DynaLab_Symbols:GS3011C -> symbols:GS3011C
Changed lines of the file:
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@@
 	)
 	(symbol
-		(lib_id "DynaLab_Symbols:GS3011C")
+		(lib_id "symbols:GS3011C")
 		(at 485.14 67.31 0)
 		(unit 1)
@@
 	)
 	(symbol
-		(lib_id "DynaLab_Symbols:GS3011C")
+		(lib_id "symbols:GS3011C")
 		(at 534.67 67.31 0)
 		(unit 1)
@@
 	)
 	(symbol
-		(lib_id "DynaLab_Symbols:GS3011C")
+		(lib_id "symbols:GS3011C")
 		(at 509.27 67.31 0)
 		(unit 1)

Commit message: update 7seg display (symbol, footprint, 3Dpackage), README
Parts:
- U5, U6, U7: footprint Footprints:GS3011A -> Footprints:GS3011
Changed lines of the file:
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@@
 			)
 		)
-		(property "Footprint" "Footprints:GS3011A"
+		(property "Footprint" "Footprints:GS3011"
 			(at 486.41 82.55 0)
 			(effects
@@
 			)
 		)
-		(property "Footprint" "Footprints:GS3011A"
+		(property "Footprint" "Footprints:GS3011"
 			(at 535.94 82.55 0)
 			(effects
@@
 			)
 		)
-		(property "Footprint" "Footprints:GS3011A"
+		(property "Footprint" "Footprints:GS3011"
 			(at 510.54 82.55 0)
 			(effects
